Commit message: [MHO] set scale to 32.8, joint type fixed, and use commas in _de.urdf

File: catkin_workspace/src/racing/urdf/racing_cart_de.urdf (robot description, URDF)
Before this commit: robot racing_cart, 2 links, 1 joints
Links:
- link map: geometry visual mesh filename=package://racing/resources/Map.dae scale=32,8 32,8 1
Joints:
- joint my_joint: type planar -> fixed

File: catkin_workspace/src/racing/urdf/racing_cart_en.urdf (robot description, URDF)
Before this commit: robot racing_cart, 2 links, 1 joints
Links:
- link map: geometry visual mesh filename=package://racing/resources/Map.dae scale=32.8 32.8 1
Joints:
- joint my_joint: type planar -> fixed
